File: LEOS-flight-computer.kicad_pcb (KiCad board)
At the start: 2 copper layers, 100 x 100 mm, 31 parts, among them J1 MicroFit_1x4, J2 MicroFit_1x4, J3 GPIO, J4 JST XH, J5 JST XH, U1 MCP2562FD, U2 MCP2518FD, U3 SAM-M8Q, Y1 40 MHz

Commit message: v2.2 with added indicator LEDs and a user button
Parts:
- added D1: Red LED, LED_SMD:LED_1206_3216Metric, F.Cu at (107.6, 92.0)
- added D2: Yellow LED, LED_SMD:LED_1206_3216Metric, F.Cu at (107.6, 95.0)
- added D3: Green LED, LED_SMD:LED_1206_3216Metric, F.Cu at (107.6, 98.0)
- added R4: 130, Resistor_SMD:R_0805_2012Metric, F.Cu at (114.0, 92.0)
- added R5: 130, Resistor_SMD:R_0805_2012Metric, F.Cu at (114.0, 95.0)
- added R6: 130, Resistor_SMD:R_0805_2012Metric, F.Cu at (114.1, 98.0)
- added SW1: User Button, Button_Switch_THT:SW_PUSH_6mm, F.Cu at (110.2, 101.8)
- R2, R3: footprint Resistor_SMD:R_0603_1608Metric -> Resistor_SMD:R_0805_2012Metric
- moved R2 1.00 mm to (163.0, 135.8)
Connections:
- J3 pad 32: GPIO12/PWM0 -> /GPIO12
- J3 pad 36: GPIO16 -> /GPIO16
- J3 pad 38: GPIO20/PCM.DIN -> /GPIO20
- J3 pad 40: GPIO21/PCM.DOUT -> /GPIO21
Routing:
- net /GPIO12: track 0.00 -> 68.6 mm, vias 0 -> 1
- net /GPIO16: track 0.00 -> 58.6 mm, vias 0 -> 1
- net /GPIO20: track 0.00 -> 58.5 mm, vias 0 -> 1
- net /GPIO21: track 0.00 -> 58.3 mm, vias 0 -> 1
- net Net-(D3-A): track 0.00 -> 4.17 mm
- net Net-(D2-A): track 0.00 -> 4.09 mm
- net Net-(D1-A): track 0.00 -> 4.09 mm
- net VDD: track 331.3 -> 332.2 mm
- net GPIO3/SCL1: track 141.8 -> 141.0 mm
Other:
- board text added: "LEOS Flight Computer Rev. 2.2"
- board text removed: "LEOS Flight Computer Rev. 2.1"
